File: dippy.kicad_pcb (KiCad board)
At the start: 2 copper layers, 3 parts, among them U1 ATmega328P-PU, U2 RFM95W-915S2, U3 MCP1700-3302E_SOT23

Commit message: update
Parts:
- added C1: 0.1u, Capacitor_THT:C_Disc_D3.0mm_W1.6mm_P2.50mm, F.Cu at (140.7, 73.7)
- added C2: 0.1u, Capacitor_THT:C_Disc_D3.0mm_W1.6mm_P2.50mm, F.Cu at (122.4, 80.3)
- added C3: 0.1u, Capacitor_THT:C_Disc_D3.0mm_W1.6mm_P2.50mm, F.Cu at (136.1, 97.2)
- added C4: 0.1u, Capacitor_THT:C_Disc_D3.0mm_W1.6mm_P2.50mm, F.Cu at (121.4, 87.9)
- added C5: 10u, Capacitor_THT:CP_Radial_D5.0mm_P2.50mm, F.Cu at (121.4, 90.9)
- added FTDI1: Conn_01x06_Male, Connector_PinHeader_2.54mm:PinHeader_1x06_P2.54mm_Horizontal, F.Cu at (123.4, 72.6)
- added H1: MountingHole, MountingHole:MountingHole_2.7mm_M2.5, F.Cu at (115.3, 67.6)
- added H2: MountingHole, MountingHole:MountingHole_2.7mm_M2.5, F.Cu at (146.8, 67.6)
- added H3: MountingHole, MountingHole:MountingHole_2.7mm_M2.5, F.Cu at (114.8, 126.5)
- added H4: MountingHole, MountingHole:MountingHole_2.7mm_M2.5, F.Cu at (146.3, 126.5)
- added J1: Conn_01x02_Female, Connector_PinSocket_2.54mm:PinSocket_1x02_P2.54mm_Vertical, F.Cu at (117.3, 86.9)
- added J2: Screw_Terminal_01x03, TerminalBlock_Phoenix:TerminalBlock_Phoenix_PT-1,5-3-3.5-H_1x03_P3.50mm_Horizontal, F.Cu at (146.8, 81.8)
- added J3: Screw_Terminal_01x04, TerminalBlock_Phoenix:TerminalBlock_Phoenix_PT-1,5-4-3.5-H_1x04_P3.50mm_Horizontal, F.Cu at (146.8, 102.6)
- added R1: 10K, Resistor_THT:R_Axial_DIN0207_L6.3mm_D2.5mm_P2.54mm_Vertical, F.Cu at (137.2, 79.8)
- added R2: 10K, Resistor_THT:R_Axial_DIN0207_L6.3mm_D2.5mm_P2.54mm_Vertical, F.Cu at (140.7, 79.8)
- added R3: 10K, Resistor_THT:R_Axial_DIN0207_L6.3mm_D2.5mm_P2.54mm_Vertical, F.Cu at (136.7, 100.1)
- added Y1: Crystal_GND2, Connector_PinSocket_2.54mm:PinSocket_1x03_P2.54mm_Vertical, F.Cu at (121.4, 102.6)
- U2: moved to B.Cu
- U3: footprint Package_TO_SOT_SMD:SOT-23 -> Package_TO_SOT_THT:TO-92L_Wide
- moved U2 22.0 mm to (137.7, 115.8), turned to 180 degrees
- moved U3 19.9 mm to (116.8, 76.2), turned to 270 degrees
Connections:
- U1 pad 1: (no net) -> Net-(C1-Pad2)
- U1 pad 10: (no net) -> Net-(U1-Pad10)
- U1 pad 13: (no net) -> D7
- U1 pad 14: (no net) -> D8
- U1 pad 2: (no net) -> RX0
- U1 pad 21: (no net) -> Net-(C3-Pad1)
- U1 pad 23: (no net) -> A0
- U1 pad 27: (no net) -> A4
- U1 pad 3: (no net) -> TX0
- U1 pad 9: (no net) -> Net-(U1-Pad9)
- U2 pad 5: (no net) -> D8
- U2 pad 6: (no net) -> D7
- U3 pad 3: (no net) -> VIN
Routing:
- net GND: track 0.00 -> 173.3 mm, vias 0 -> 4
- net VCC: track 0.00 -> 144.5 mm, vias 0 -> 6
- net (no net): track 0.00 -> 45.3 mm, vias 0 -> 2
- net SCK: track 0.00 -> 27.2 mm
- net D7: track 0.00 -> 26.7 mm
- net A0: track 0.00 -> 22.5 mm, vias 0 -> 2
- net VIN: track 0.00 -> 21.2 mm
- net MOSI: track 0.00 -> 20.3 mm
- net MISO: track 0.00 -> 18.9 mm
- net D8: track 0.00 -> 18.2 mm
- net Net-(C1-Pad2): track 0.00 -> 18.2 mm, vias 0 -> 2
- net TX0: track 0.00 -> 16.0 mm
- net A4: track 0.00 -> 15.5 mm
- net RX0: track 0.00 -> 12.7 mm
- net Net-(U1-Pad9): track 0.00 -> 5.21 mm
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Other:
- board outline added: 41.7 x 70.1 mm

Commit message: update
Connections:
- U1 pad 12: (no net) -> D6
- U1 pad 5: (no net) -> D3
- U2 pad 14: (no net) -> D3
- U2 pad 15: (no net) -> D6
Routing:
- net (no net): track 45.3 -> 4.68 mm
- net D3: track 0.00 -> 40.2 mm, vias 0 -> 2
- net D6: track 0.00 -> 16.8 mm
- net VCC: track 144.5 -> 148.2 mm

Commit message: update
Parts:
- removed H1, H3: MountingHole, MountingHole:MountingHole_2.7mm_M2.5
- added R4: 100K, Resistor_THT:R_Axial_DIN0207_L6.3mm_D2.5mm_P7.62mm_Horizontal, F.Cu at (128.3, 72.3)
- added R5: 100K, Resistor_THT:R_Axial_DIN0207_L6.3mm_D2.5mm_P2.54mm_Vertical, F.Cu at (136.7, 77.6)
- C1: footprint Capacitor_THT:C_Disc_D3.0mm_W1.6mm_P2.50mm -> Capacitor_THT:C_Disc_D4.7mm_W2.5mm_P5.00mm
- R1: footprint Resistor_THT:R_Axial_DIN0207_L6.3mm_D2.5mm_P2.54mm_Vertical -> Resistor_THT:R_Axial_DIN0207_L6.3mm_D2.5mm_P5.08mm_Vertical
- U1: value ATmega328P-PU -> ATmega328P-PU-C
- Y1: value Crystal_GND2 -> Crystal; footprint Connector_PinSocket_2.54mm:PinSocket_1x03_P2.54mm_Vertical -> Crystal:Resonator-2Pin_W10.0mm_H5.0mm
- moved R1 17.2 mm to (120.4, 75.9), turned to 0 degrees
- moved C1 15.9 mm to (124.8, 72.9), turned to 180 degrees
- moved R2 7.19 mm to (136.9, 85.9)
- moved FTDI1 6.36 mm to (123.2, 66.3)
- moved J2 5.64 mm to (142.2, 85.1)
- moved J3 4.86 mm to (142.2, 101.0)
- moved C5 3.69 mm to (121.5, 94.6)
- moved R3 2.30 mm to (136.9, 102.4), turned to 90 degrees
- moved H2 1.76 mm to (146.0, 66.0)
- moved Y1 0.77 mm to (121.3, 101.9), turned to 270 degrees
- moved H4 0.58 mm to (146.0, 126.0)
- moved C3 0.28 mm to (136.4, 97.0)
Connections:
- FTDI1 pad 6: Net-(C1-Pad1) -> Net-(C1-Pad2)
- J2 pad 2: A4 -> A2
- J3 pad 1: VCC -> GND
- J3 pad 2: A0 -> VCC
- J3 pad 3: (no net) -> A0
- J3 pad 4: GND -> A1
- R1 pad 2: Net-(C1-Pad2) -> Net-(C1-Pad1)
- R2 pad 2: A4 -> A2
- U1 pad 1: Net-(C1-Pad2) -> Net-(C1-Pad1)
- U1 pad 24: (no net) -> A1
- U1 pad 25: (no net) -> A2
- U1 pad 27: A4 -> (no net)
- U1 pad 28: (no net) -> A5
- Y1 pad 1: Net-(U1-Pad10) -> Net-(U1-Pad9)
- Y1 pad 2: GND -> Net-(U1-Pad10)
Routing:
- net VCC: track 148.2 -> 207.1 mm, vias 6 -> 4
- net GND: track 173.3 -> 226.8 mm, vias 4 -> 9
- net A4: track 15.5 -> 0.00 mm
- net A2: track 0.00 -> 15.0 mm
- net A5: track 0.00 -> 12.1 mm
- net A1: track 0.00 -> 9.28 mm
- net Net-(C1-Pad2): track 18.2 -> 26.9 mm, vias 2 -> 0
- net VIN: track 21.2 -> 29.9 mm
- net (no net): track 4.68 -> 11.0 mm, vias 2 -> 4
- net TX0: track 16.0 -> 22.4 mm
- net RX0: track 12.7 -> 19.0 mm
- net A0: track 22.5 -> 18.9 mm, vias 2 -> 0
- net MISO: track 18.9 -> 22.0 mm, vias 0 -> 1
- net Net-(U1-Pad10): track 4.48 -> 7.12 mm
- net Net-(C1-Pad1): track 4.99 -> 6.85 mm
Other:
- board size 41.7 x 70.1 mm -> 43.1 x 72.6 mm

Commit message: update
Parts:
- moved FTDI1 2.16 mm to (123.1, 68.5)
- moved H2 1.00 mm to (146.0, 67.0)
- moved H4 1.00 mm to (146.0, 127.0)
- moved R4 0.97 mm to (127.4, 72.6)
Routing:
- net VCC: track 207.1 -> 157.0 mm, vias 4 -> 7
- net GND: track 226.8 -> 222.7 mm, vias 9 -> 7
- net RX0: track 19.0 -> 16.2 mm
- net TX0: track 22.4 -> 20.1 mm
- net VIN: track 29.9 -> 28.0 mm
- net A5: track 12.1 -> 11.4 mm
Other:
- board size 43.1 x 72.6 mm -> 40.6 x 69.6 mm

Commit message: update
Parts:
- moved H4 2.91 mm to (146.6, 129.9)
- moved H2 0.85 mm to (145.6, 67.8)
Routing:
- net VCC: track 157.0 -> 277.3 mm, vias 7 -> 9
- net GND: track 222.7 -> 226.4 mm
Other:
- board size 40.6 x 69.6 mm -> 42.2 x 69.9 mm
Changed lines of the file:
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@@
-(kicad_pcb (version 20171130) (host pcbnew 5.1.5-52549c5~84~ubuntu18.04.1)
+(kicad_pcb (version 20171130) (host pcbnew 5.1.2-f72e74a~84~ubuntu18.04.1)
   (general
     (thickness 1.6)
     (drawings 4)
-    (tracks 329)
+    (tracks 353)
     (zones 0)
     (modules 20)
@@
     (add_net A1)
     (add_net A2)
-    (add_net A3)
-    (add_net A4)
     (add_net A5)
-    (add_net D2)
     (add_net D3)
-    (add_net D4)
-    (add_net D5)
     (add_net D6)
     (add_net D7)
@@
     (add_net "Net-(C1-Pad2)")
     (add_net "Net-(C3-Pad1)")
-    (add_net "Net-(FTDI1-Pad2)")
     (add_net "Net-(U1-Pad10)")
     (add_net "Net-(U1-Pad9)")
-    (add_net "Net-(U2-Pad11)")
-    (add_net "Net-(U2-Pad12)")
-    (add_net "Net-(U2-Pad16)")
-    (add_net "Net-(U2-Pad7)")
-    (add_net "Net-(U2-Pad9)")
     (add_net RX0)
     (add_net SCK)
@@
   )
   (module MountingHole:MountingHole_2.7mm_M2.5 (layer F.Cu)
-    (at 146 127)
+    (at 146.558 129.8575)
     (descr "Mounting Hole 2.7mm, no annular, M2.5")
     (tags "mounting hole 2.7mm no annular m2.5")
@@
   )
   (module MountingHole:MountingHole_2.7mm_M2.5 (layer F.Cu)
-    (at 146 67)
+    (at 145.6055 67.7545)
     (descr "Mounting Hole 2.7mm, no annular, M2.5")
     (tags "mounting hole 2.7mm no annular m2.5")
@@
     )
   )
-  (gr_line (start 150.241 62.484) (end 109.601 62.484) (layer Edge.Cuts) (width 0.05))
-  (gr_line (start 109.601 132.08) (end 109.601 62.484) (layer Edge.Cuts) (width 0.05))
-  (gr_line (start 150.241 132.08) (end 109.601 132.08) (layer Edge.Cuts) (width 0.05))
-  (gr_line (start 150.241 132.08) (end 150.241 62.484) (layer Edge.Cuts) (width 0.05))
+  (gr_line (start 107.8865 64.1985) (end 107.8865 134.112) (layer Edge.Cuts) (width 0.05))
+  (gr_line (start 150.114 134.112) (end 107.8865 134.112) (layer Edge.Cuts) (width 0.05))
+  (gr_line (start 150.114 64.1985) (end 150.114 134.112) (layer Edge.Cuts) (width 0.05))
+  (gr_line (start 107.8865 64.1985) (end 150.114 64.1985) (layer Edge.Cuts) (width 0.05))
   (via (at 135.636 109.728) (size 1.5) (drill 0.75) (layers F.Cu B.Cu) (net 0))
   (segment (start 133.35 109.855) (end 135.509 109.855) (width 1) (layer B.Cu) (net 0))
@@
   (segment (start 118.364 98.933) (end 113.809198 98.933) (width 1) (layer F.Cu) (net 3))
   (via (at 119.761 68.58) (size 1.5) (drill 0.75) (layers F.Cu B.Cu) (net 3))
-  (segment (start 116.84 75.692) (end 116.84 76.2) (width 1) (layer B.Cu) (net 3))
   (segment (start 145.542 74.422) (end 143.383 72.263) (width 1) (layer B.Cu) (net 3))
   (segment (start 143.383 72.263) (end 140.843 72.263) (width 1) (layer B.Cu) (net 3))
@@
   (segment (start 145.542 83.988) (end 145.542 74.422) (width 1) (layer B.Cu) (net 3))
   (segment (start 140.843 72.263) (end 138.049 75.057) (width 1) (layer B.Cu) (net 3))
-  (via (at 116.84 72.644) (size 1.5) (drill 0.75) (layers F.Cu B.Cu) (net 3))
-  (segment (start 116.84 76.2) (end 116.84 72.644) (width 1) (layer B.Cu) (net 3))
   (segment (start 119.888 68.453) (end 119.761 68.58) (width 1) (layer B.Cu) (net 3))
   (segment (start 123.063 68.453) (end 119.888 68.453) (width 1) (layer B.Cu) (net 3))
-  (segment (start 116.84 71.501) (end 119.761 68.58) (width 1) (layer F.Cu) (net 3))
-  (segment (start 116.84 72.644) (end 116.84 71.501) (width 1) (layer F.Cu) (net 3))
+  (segment (start 116.84 76.2) (end 116.84 75.946) (width 1) (layer B.Cu) (net 3))
+  (segment (start 116.84 76.2) (end 116.84 75.819) (width 1) (layer B.Cu) (net 3))
+  (segment (start 116.84 75.819) (end 116.332 75.311) (width 1) (layer B.Cu) (net 3))
+  (segment (start 116.332 75.311) (end 116.332 72.517) (width 1) (layer B.Cu) (net 3))
+  (via (at 115.316 68.5165) (size 1.5) (drill 0.75) (layers F.Cu B.Cu) (net 3))
+  (segment (start 116.332 72.517) (end 115.316 71.501) (width 1) (layer B.Cu) (net 3))
+  (segment (start 115.316 71.501) (end 115.316 68.5165) (width 1) (layer B.Cu) (net 3))
+  (segment (start 119.6975 68.5165) (end 119.761 68.58) (width 1) (layer F.Cu) (net 3))
+  (segment (start 115.316 68.5165) (end 119.6975 68.5165) (width 1) (layer F.Cu) (net 3))
   (segment (start 125.73 76.2) (end 125.476 75.946) (width 1) (layer B.Cu) (net 4))
   (segment (start 125.73 79.375) (end 125.73 76.2) (width 1) (layer B.Cu) (net 4))
@@
   (segment (start 143.891 72.771) (end 142.24 74.422) (width 1) (layer F.Cu) (net 5))
   (segment (start 147.193 72.771) (end 143.891 72.771) (width 1) (layer F.Cu) (net 5))
+  (segment (start 145.034 106.426) (end 145.034 114.6175) (width 1) (layer B.Cu) (net 5))
+  (segment (start 145.034 114.6175) (end 145.161 114.7445) (width 1) (layer B.Cu) (net 5))
+  (segment (start 145.161 114.7445) (end 145.161 120.5865) (width 1) (layer B.Cu) (net 5))
+  (segment (start 145.161 120.5865) (end 142.621 123.1265) (width 1) (layer B.Cu) (net 5))
+  (segment (start 142.621 123.1265) (end 142.621 129.54) (width 1) (layer B.Cu) (net 5))
+  (segment (start 142.621 129.54) (end 139.954 132.207) (width 1) (layer B.Cu) (net 5))
+  (segment (start 139.954 132.207) (end 117.094 132.207) (width 1) (layer B.Cu) (net 5))
+  (segment (start 112.2045 127.3175) (end 112.2045 127.254) (width 1) (layer B.Cu) (net 5))
+  (segment (start 117.094 132.207) (end 112.2045 127.3175) (width 1) (layer B.Cu) (net 5))
+  (segment (start 112.2045 127.254) (end 110.2995 125.349) (width 1) (layer B.Cu) (net 5))
+  (segment (start 110.2995 125.349) (end 110.2995 77.9145) (width 1) (layer B.Cu) (net 5))
+  (segment (start 110.2995 77.9145) (end 110.2995 77.7875) (width 1) (layer B.Cu) (net 5))
+  (via (at 113.9825 74.168) (size 1.5) (drill 0.75) (layers F.Cu B.Cu) (net 5))
+  (segment (start 110.2995 77.7875) (end 113.919 74.168) (width 1) (layer B.Cu) (net 5))
+  (via (at 118.491 74.6125) (size 1.5) (drill 0.75) (layers F.Cu B.Cu) (net 5))
+  (segment (start 114.8715 74.168) (end 118.0465 74.168) (width 1) (layer F.Cu) (net 5))
+  (segment (start 118.0465 74.168) (end 118.491 74.6125) (width 1) (layer F.Cu) (net 5))
+  (segment (start 119.0625 74.6125) (end 120.396 75.946) (width 1) (layer B.Cu) (net 5))
+  (segment (start 118.491 74.6125) (end 119.0625 74.6125) (width 1) (layer B.Cu) (net 5))
+  (segment (start 114.8715 74.168) (end 113.9825 74.168) (width 1) (layer F.Cu) (net 5))
   (segment (start 129.032 104.648) (end 131.445 102.235) (width 1) (layer B.Cu) (net 6))
   (segment (start 137.668 121.824) (end 135.668 121.824) (width 1) (layer B.Cu) (net 6))

Commit message: update
Parts:
- moved H2 1.42 mm to (147.0, 68.0)
- moved H4 0.46 mm to (147.0, 130.0)
Other:
- board size 42.2 x 69.9 mm -> 43.6 x 69.9 mm
Changed lines of the file:
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@@
   (general
     (thickness 1.6)
-    (drawings 4)
+    (drawings 6)
     (tracks 353)
     (zones 0)
@@
   )
   (module MountingHole:MountingHole_2.7mm_M2.5 (layer F.Cu)
-    (at 146.558 129.8575)
+    (at 147 130)
     (descr "Mounting Hole 2.7mm, no annular, M2.5")
     (tags "mounting hole 2.7mm no annular m2.5")
@@
   )
   (module MountingHole:MountingHole_2.7mm_M2.5 (layer F.Cu)
-    (at 145.6055 67.7545)
+    (at 147 68)
     (descr "Mounting Hole 2.7mm, no annular, M2.5")
     (tags "mounting hole 2.7mm no annular m2.5")
@@
     )
   )
+  (gr_line (start 150.114 64.1985) (end 151.4475 64.1985) (layer Edge.Cuts) (width 0.05))
+  (gr_line (start 151.4475 134.112) (end 150.114 134.112) (layer Edge.Cuts) (width 0.05))
+  (gr_line (start 151.4475 64.1985) (end 151.4475 134.112) (layer Edge.Cuts) (width 0.05))
   (gr_line (start 107.8865 64.1985) (end 107.8865 134.112) (layer Edge.Cuts) (width 0.05))
   (gr_line (start 150.114 134.112) (end 107.8865 134.112) (layer Edge.Cuts) (width 0.05))
-  (gr_line (start 150.114 64.1985) (end 150.114 134.112) (layer Edge.Cuts) (width 0.05))
   (gr_line (start 107.8865 64.1985) (end 150.114 64.1985) (layer Edge.Cuts) (width 0.05))
   (via (at 135.636 109.728) (size 1.5) (drill 0.75) (layers F.Cu B.Cu) (net 0))
