File: ver1/dippy.kicad_pcb (KiCad board)
At the start: 2 copper layers, 40.6 x 69.6 mm, 20 parts, among them J1 Conn_01x02_Female, J2 Screw_Terminal_01x03, J3 Screw_Terminal_01x04, U1 ATmega328P-PU-C, U2 RFM95W-915S2, U3 MCP1700-3302E_SOT23, Y1 Crystal

Commit message: update
Parts:
- moved H4 3.16 mm to (147.0, 130.0)
- moved H2 1.41 mm to (147.0, 68.0)
Routing:
- net VCC: track 157.0 -> 277.3 mm, vias 7 -> 9
- net GND: track 222.7 -> 226.4 mm
Other:
- board size 40.6 x 69.6 mm -> 43.6 x 69.9 mm
Changed lines of the file:
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@@
-(kicad_pcb (version 20171130) (host pcbnew 5.1.5-52549c5~84~ubuntu18.04.1)
+(kicad_pcb (version 20171130) (host pcbnew 5.1.2-f72e74a~84~ubuntu18.04.1)
   (general
     (thickness 1.6)
-    (drawings 4)
-    (tracks 329)
+    (drawings 6)
+    (tracks 353)
     (zones 0)
     (modules 20)
@@
     (add_net A1)
     (add_net A2)
-    (add_net A3)
-    (add_net A4)
     (add_net A5)
-    (add_net D2)
     (add_net D3)
-    (add_net D4)
-    (add_net D5)
     (add_net D6)
     (add_net D7)
@@
     (add_net "Net-(C1-Pad2)")
     (add_net "Net-(C3-Pad1)")
-    (add_net "Net-(FTDI1-Pad2)")
     (add_net "Net-(U1-Pad10)")
     (add_net "Net-(U1-Pad9)")
-    (add_net "Net-(U2-Pad11)")
-    (add_net "Net-(U2-Pad12)")
-    (add_net "Net-(U2-Pad16)")
-    (add_net "Net-(U2-Pad7)")
-    (add_net "Net-(U2-Pad9)")
     (add_net RX0)
     (add_net SCK)
@@
   )
   (module MountingHole:MountingHole_2.7mm_M2.5 (layer F.Cu)
-    (at 146 127)
+    (at 147 130)
     (descr "Mounting Hole 2.7mm, no annular, M2.5")
     (tags "mounting hole 2.7mm no annular m2.5")
@@
   )
   (module MountingHole:MountingHole_2.7mm_M2.5 (layer F.Cu)
-    (at 146 67)
+    (at 147 68)
     (descr "Mounting Hole 2.7mm, no annular, M2.5")
     (tags "mounting hole 2.7mm no annular m2.5")
@@
     )
   )
-  (gr_line (start 150.241 62.484) (end 109.601 62.484) (layer Edge.Cuts) (width 0.05))
-  (gr_line (start 109.601 132.08) (end 109.601 62.484) (layer Edge.Cuts) (width 0.05))
-  (gr_line (start 150.241 132.08) (end 109.601 132.08) (layer Edge.Cuts) (width 0.05))
-  (gr_line (start 150.241 132.08) (end 150.241 62.484) (layer Edge.Cuts) (width 0.05))
+  (gr_line (start 150.114 64.1985) (end 151.4475 64.1985) (layer Edge.Cuts) (width 0.05))
+  (gr_line (start 151.4475 134.112) (end 150.114 134.112) (layer Edge.Cuts) (width 0.05))
+  (gr_line (start 151.4475 64.1985) (end 151.4475 134.112) (layer Edge.Cuts) (width 0.05))
+  (gr_line (start 107.8865 64.1985) (end 107.8865 134.112) (layer Edge.Cuts) (width 0.05))
+  (gr_line (start 150.114 134.112) (end 107.8865 134.112) (layer Edge.Cuts) (width 0.05))
+  (gr_line (start 107.8865 64.1985) (end 150.114 64.1985) (layer Edge.Cuts) (width 0.05))
   (via (at 135.636 109.728) (size 1.5) (drill 0.75) (layers F.Cu B.Cu) (net 0))
   (segment (start 133.35 109.855) (end 135.509 109.855) (width 1) (layer B.Cu) (net 0))
@@
   (segment (start 118.364 98.933) (end 113.809198 98.933) (width 1) (layer F.Cu) (net 3))
   (via (at 119.761 68.58) (size 1.5) (drill 0.75) (layers F.Cu B.Cu) (net 3))
-  (segment (start 116.84 75.692) (end 116.84 76.2) (width 1) (layer B.Cu) (net 3))
   (segment (start 145.542 74.422) (end 143.383 72.263) (width 1) (layer B.Cu) (net 3))
   (segment (start 143.383 72.263) (end 140.843 72.263) (width 1) (layer B.Cu) (net 3))
@@
   (segment (start 145.542 83.988) (end 145.542 74.422) (width 1) (layer B.Cu) (net 3))
   (segment (start 140.843 72.263) (end 138.049 75.057) (width 1) (layer B.Cu) (net 3))
-  (via (at 116.84 72.644) (size 1.5) (drill 0.75) (layers F.Cu B.Cu) (net 3))
-  (segment (start 116.84 76.2) (end 116.84 72.644) (width 1) (layer B.Cu) (net 3))
   (segment (start 119.888 68.453) (end 119.761 68.58) (width 1) (layer B.Cu) (net 3))
   (segment (start 123.063 68.453) (end 119.888 68.453) (width 1) (layer B.Cu) (net 3))
-  (segment (start 116.84 71.501) (end 119.761 68.58) (width 1) (layer F.Cu) (net 3))
-  (segment (start 116.84 72.644) (end 116.84 71.501) (width 1) (layer F.Cu) (net 3))
+  (segment (start 116.84 76.2) (end 116.84 75.946) (width 1) (layer B.Cu) (net 3))
+  (segment (start 116.84 76.2) (end 116.84 75.819) (width 1) (layer B.Cu) (net 3))
+  (segment (start 116.84 75.819) (end 116.332 75.311) (width 1) (layer B.Cu) (net 3))
+  (segment (start 116.332 75.311) (end 116.332 72.517) (width 1) (layer B.Cu) (net 3))
+  (via (at 115.316 68.5165) (size 1.5) (drill 0.75) (layers F.Cu B.Cu) (net 3))
+  (segment (start 116.332 72.517) (end 115.316 71.501) (width 1) (layer B.Cu) (net 3))
+  (segment (start 115.316 71.501) (end 115.316 68.5165) (width 1) (layer B.Cu) (net 3))
+  (segment (start 119.6975 68.5165) (end 119.761 68.58) (width 1) (layer F.Cu) (net 3))
+  (segment (start 115.316 68.5165) (end 119.6975 68.5165) (width 1) (layer F.Cu) (net 3))
   (segment (start 125.73 76.2) (end 125.476 75.946) (width 1) (layer B.Cu) (net 4))
   (segment (start 125.73 79.375) (end 125.73 76.2) (width 1) (layer B.Cu) (net 4))
@@
   (segment (start 143.891 72.771) (end 142.24 74.422) (width 1) (layer F.Cu) (net 5))
   (segment (start 147.193 72.771) (end 143.891 72.771) (width 1) (layer F.Cu) (net 5))
+  (segment (start 145.034 106.426) (end 145.034 114.6175) (width 1) (layer B.Cu) (net 5))
+  (segment (start 145.034 114.6175) (end 145.161 114.7445) (width 1) (layer B.Cu) (net 5))
+  (segment (start 145.161 114.7445) (end 145.161 120.5865) (width 1) (layer B.Cu) (net 5))
+  (segment (start 145.161 120.5865) (end 142.621 123.1265) (width 1) (layer B.Cu) (net 5))
+  (segment (start 142.621 123.1265) (end 142.621 129.54) (width 1) (layer B.Cu) (net 5))
+  (segment (start 142.621 129.54) (end 139.954 132.207) (width 1) (layer B.Cu) (net 5))
+  (segment (start 139.954 132.207) (end 117.094 132.207) (width 1) (layer B.Cu) (net 5))
+  (segment (start 112.2045 127.3175) (end 112.2045 127.254) (width 1) (layer B.Cu) (net 5))
+  (segment (start 117.094 132.207) (end 112.2045 127.3175) (width 1) (layer B.Cu) (net 5))
+  (segment (start 112.2045 127.254) (end 110.2995 125.349) (width 1) (layer B.Cu) (net 5))
+  (segment (start 110.2995 125.349) (end 110.2995 77.9145) (width 1) (layer B.Cu) (net 5))
+  (segment (start 110.2995 77.9145) (end 110.2995 77.7875) (width 1) (layer B.Cu) (net 5))
+  (via (at 113.9825 74.168) (size 1.5) (drill 0.75) (layers F.Cu B.Cu) (net 5))
+  (segment (start 110.2995 77.7875) (end 113.919 74.168) (width 1) (layer B.Cu) (net 5))
+  (via (at 118.491 74.6125) (size 1.5) (drill 0.75) (layers F.Cu B.Cu) (net 5))
+  (segment (start 114.8715 74.168) (end 118.0465 74.168) (width 1) (layer F.Cu) (net 5))
+  (segment (start 118.0465 74.168) (end 118.491 74.6125) (width 1) (layer F.Cu) (net 5))
+  (segment (start 119.0625 74.6125) (end 120.396 75.946) (width 1) (layer B.Cu) (net 5))
+  (segment (start 118.491 74.6125) (end 119.0625 74.6125) (width 1) (layer B.Cu) (net 5))
+  (segment (start 114.8715 74.168) (end 113.9825 74.168) (width 1) (layer F.Cu) (net 5))
   (segment (start 129.032 104.648) (end 131.445 102.235) (width 1) (layer B.Cu) (net 6))
   (segment (start 137.668 121.824) (end 135.668 121.824) (width 1) (layer B.Cu) (net 6))
